File: 2024_C_AV_HW-TSE.kicad_sch (KiCad schematic)
At the start: 35 parts, among them J1 Spine Connector, J2 I2C Bypass, U1 LT3960, U2 Teensy4.0

Commit message: uart
Parts:
- added D?: TPD2E1B06DRLR, TPD2E1B06DRLR:SOTFL50P160X60-6N, symbol TPD2E1B06DRLR:TPD2E1B06DRLR
- added J?: USART Bypass, Connector_PinHeader_2.00mm:PinHeader_1x02_P2.00mm_Vertical, symbol Connector_Generic:Conn_01x02
- added R? (x2): 0R, Resistor_SMD:R_0805_2012Metric_Pad1.20x1.40mm_HandSolder, symbol Device:R
Connections:
- net GND: now also D?.2 (IOB1), D?.5 (IOA2)
- net TX_Te: now reaches U2.10 (8_TX2_IN1)
- net TX_Te: now also R?.2
- net RX_Te: now reaches U2.9 (7_RX2_OUT1A)
- net RX_Te: now also R?.2
- new net RX_Ta: D?.3 (NC_1), D?.4 (IOB2), J?.1 (Pin_1), R?.1
- new net TX_Ta: D?.1 (IOA1), D?.6 (NC_2), J?.2 (Pin_2), R?.1
- no-connect marks 41 -> 39
Other:
- note added: "USART Conenctor"
- note added: "USART POKA-YOKE"
