File: 2024_C_AV_HW-TSE.kicad_pcb (KiCad board)
At the start: 2 copper layers, 35 parts, among them J1 Spine Connector, J2 I2C Bypass, U1 LT3960, U2 Teensy4.0

Commit message: layout
Parts:
- added D8: TPD2E1B06DRLR, TPD2E1B06DRLR:SOTFL50P160X60-6N, F.Cu at (83.2, 37.5)
- added J3: USART Bypass, Connector_PinHeader_2.00mm:PinHeader_1x02_P2.00mm_Vertical, F.Cu at (79.4, 32.1)
- added R10: 0R, Resistor_SMD:R_0805_2012Metric_Pad1.20x1.40mm_HandSolder, F.Cu at (83.8, 34.5)
- added R9: 0R, Resistor_SMD:R_0805_2012Metric_Pad1.20x1.40mm_HandSolder, F.Cu at (83.8, 31.5)
Connections:
- U2 pad 10: unconnected-(U2-8_TX2_IN1-Pad10) -> /TX_Te
- U2 pad 9: unconnected-(U2-7_RX2_OUT1A-Pad9) -> /RX_Te
